File: so2rminiplus.kicad_pcb (KiCad board)
At the start: 2 copper layers, 93 x 92 mm, 73 parts, among them J1 STX-3000, J10 Conn_01x10_Pin, J11 Conn_01x03_Pin, J12 STX-3000, J13 STX-3000, J14 Conn_01x02_Pin, J15 Conn_01x02_Pin, J2 STX-3000, J3 STX-3000, J4 STX-3000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

Commit message: Make assembly layer more readable.
Parts:
- D4: value LEDs Wuerth 150141M173100 -> LED
- D5: value LED_Dual_AAKK -> LED

Commit message: Fix swapped pins 4 and 7 on relay K3.
Thanks to Peter, LA7WRA / LZ1VPC for finding this!
Parts:
- D4: value LED -> LEDs Wuerth 150141RV731
- D5: value LED -> LED_Dual_AAKK
Connections:
- K3 pad 4: Net-(J14-Pin_1) -> Net-(J3-PadS)
- K3 pad 7: Net-(J3-PadS) -> Net-(J14-Pin_1)
Routing:
- net Net-(J14-Pin_1): track 9.11 -> 17.2 mm
- net Net-(J3-PadS): track 27.4 -> 29.9 mm, vias 0 -> 2
Other:
- board text added: "PCB Rev 2c - 2025-12-28"
- board text removed: "PCB Rev 2 - 2025-08-24"
